File: Spartan 6 FPGA Board/Spartan 6 FPGA Board/Power_supply.sch.kicad_sch (KiCad schematic)
At the start: 75 parts, among them J2 XT30PW-M, Q1 GSFC02A05, Q2 GSFC02A05, Q3 GSFC02A05, Q4 NPN, U18 AP7363-33D-13, U19 AP7363-25D-13, U3 TPS562201DDCR, U4 TPS562201DDCR, U5 TPS562201DDCR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

Commit message: Add files via upload
Updated files with new libraries
Parts:
- TP1, TP3: footprint TestPoint:TestPoint_Pad_D1.0mm -> Personal-Library:TestPoint_Pad_D1.0mm
Changed lines of the file:
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@@
 			)
 		)
-		(property "Footprint" "TestPoint:TestPoint_Pad_D1.0mm"
+		(property "Footprint" "Personal-Library:TestPoint_Pad_D1.0mm"
 			(at 132.08 186.69 0)
 			(effects
@@
 			)
 		)
-		(property "Footprint" "TestPoint:TestPoint_Pad_D1.0mm"
+		(property "Footprint" "Personal-Library:TestPoint_Pad_D1.0mm"
 			(at 132.08 181.61 0)
 			(effects
