File: Spartan 6 FPGA Board/Spartan 6 FPGA Board/Spartan 6 FPGA Board.kicad_pcb (KiCad board)
At the start: 4 copper layers, 99 x 99 mm, 261 parts, among them J1 USB_B_Micro, J2 XT30PW-M, J3 Left Side, J4 RIght Side, Q1 GSFC02A05, Q2 GSFC02A05, Q3 GSFC02A05, Q4 NPN, SW5 RES_FLASH, U1 XC6SLX9-2TQG144C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

Commit message: Add files via upload
Updated files with new libraries
Parts:
- TP1, TP2, TP3, TP4, TP5, TP6, TP7: footprint TestPoint:TestPoint_Pad_D1.0mm -> Personal-Library:TestPoint_Pad_D1.0mm
Changed lines of the file:
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@@
 		)
 	)
-	(footprint "TestPoint:TestPoint_Pad_D1.0mm"
+	(footprint "Personal-Library:TestPoint_Pad_D1.0mm"
 		(layer "F.Cu")
 		(at 132.34416 113.67008)
@@
 			)
 		)
-		(property "Field5" "TMS"
-			(at 0.03048 2.21488 90)
+		(property "Field4" "TMS"
+			(at 0 2.38992 90)
 			(unlocked yes)
 			(layer "F.SilkS")
@@
 			(layer "F.CrtYd")
 		)
-		(fp_text user "${REFERENCE}"
-			(at 0 -1.45 0)
-			(layer "F.Fab")
-			(effects
-				(font
-					(size 1 1)
-					(thickness 0.15)
-				)
-			)
-		)
 		(pad "1" smd circle
 			(at 0 0)
@@
 		)
 	)
-	(footprint "TestPoint:TestPoint_Pad_D1.0mm"
+	(footprint "Personal-Library:TestPoint_Pad_D1.0mm"
 		(layer "F.Cu")
 		(at 130.1242 113.68024)
@@
 			)
 		)
-		(property "Field5" "TDO"
-			(at 0.01524 2.40284 90)
+		(property "Field4" "TDO"
+			(at 0 2.36976 90)
 			(unlocked yes)
 			(layer "F.SilkS")
@@
 			(layer "F.CrtYd")
 		)
-		(fp_text user "${REFERENCE}"
-			(at 0 -1.45 0)
-			(layer "F.Fab")
-			(effects
-				(font
-					(size 1 1)
-					(thickness 0.15)
-				)
-			)
-		)
 		(pad "1" smd circle
 			(at 0 0)
@@
 		)
 	)
-	(footprint "TestPoint:TestPoint_Pad_D1.0mm"
+	(footprint "Personal-Library:TestPoint_Pad_D1.0mm"
 		(layer "F.Cu")
 		(at 127.56896 113.70056)
@@
 			)
 		)
-		(property "Field5" "TCK"
-			(at 0.03048 2.30124 90)
+		(property "Field4" "TCK"
+			(at 0 2.26944 90)
 			(unlocked yes)
 			(layer "F.SilkS")
@@
 			(layer "F.CrtYd")
 		)
-		(fp_text user "${REFERENCE}"
-			(at 0 -1.45 0)
-			(layer "F.Fab")
-			(effects
-				(font
-					(size 1 1)
-					(thickness 0.15)
-				)
-			)
-		)
 		(pad "1" smd circle
 			(at 0 0)
@@
 		)
 	)
-	(footprint "TestPoint:TestPoint_Pad_D1.0mm"
+	(footprint "Personal-Library:TestPoint_Pad_D1.0mm"
 		(layer "F.Cu")
 		(at 125.21692 113.69548)
@@
 			)
 		)
-		(property "Field5" "TDI"
-			(at -0.09652 2.40792 90)
+		(property "Field4" "TDI"
+			(at 0 2.11452 90)
 			(unlocked yes)
 			(layer "F.SilkS")
@@
 			(layer "F.CrtYd")
 		)
-		(fp_text user "${REFERENCE}"
-			(at 0 -1.45 0)
-			(layer "F.Fab")
-			(effects
-				(font
-					(size 1 1)
-					(thickness 0.15)
-				)
-			)
-		)
 		(pad "1" smd circle
 			(at 0 0)
@@
 		)
 	)
-	(footprint "TestPoint:TestPoint_Pad_D1.0mm"
+	(footprint "Personal-Library:TestPoint_Pad_D1.0mm"
 		(layer "B.Cu")
 		(at 154.60472 66.68008 180)
@@
 			)
 		)
-		(property "Field5" "+3.3V"
-			(at -0.18288 1.524 0)
+		(property "Field4" "+3.3V"
+			(at -0.04528 1.60008 0)
 			(unlocked yes)
 			(layer "B.SilkS")
@@
 			(layer "B.CrtYd")
 		)
-		(fp_text user "${REFERENCE}"
-			(at 0 1.45 0)
-			(layer "B.Fab")
-			(effects
-				(font
-					(size 1 1)
-					(thickness 0.15)
-				)
-				(justify mirror)
-			)
-		)
 		(pad "1" smd circle
 			(at 0 0 180)
@@
 		)
 	)
-	(footprint "TestPoint:TestPoint_Pad_D1.0mm"
+	(footprint "Personal-Library:TestPoint_Pad_D1.0mm"
 		(layer "B.Cu")
 		(at 175.26508 65.85712 180)
@@
 			)
 		)
-		(property "Field5" "VCCINT"
-			(at 0.08128 -1.59512 0)
+		(property "Field4" "VCCINT"
+			(at 0.03508 -1.72288 0)
 			(unlocked yes)
 			(layer "B.SilkS")
@@
 		)
 	)
-	(footprint "TestPoint:TestPoint_Pad_D1.0mm"
+	(footprint "Personal-Library:TestPoint_Pad_D1.0mm"
 		(layer "B.Cu")
 		(at 165.59276 54.51348 180)
@@
 			)
 		)
-		(property "Field5" "VCCO"
-			(at 0.14732 1.46812 0)
+		(property "Field4" "VCCO"
+			(at -0.01724 1.55348 0)
 			(unlocked yes)
 			(layer "B.SilkS")
@@
 			(layer "B.CrtYd")
 		)
-		(fp_text user "${REFERENCE}"
-			(at 0 1.45 0)
-			(layer "B.Fab")
-			(effects
-				(font
-					(size 1 1)
-					(thickness 0.15)
-				)
-				(justify mirror)
-			)
-		)
 		(pad "1" smd circle
