File: Spartan 6 FPGA Board/Spartan 6 FPGA Board/untitled.kicad_sch (KiCad schematic)
At the start: 50 parts, among them U1 XC6SLX9-2TQG144C

Commit message: Add files via upload
Updated files with new libraries
Parts:
- TP2, TP4, TP5, TP6, TP7: footprint TestPoint:TestPoint_Pad_D1.0mm -> Personal-Library:TestPoint_Pad_D1.0mm
Changed lines of the file:
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@@
 			)
 		)
-		(property "Footprint" "TestPoint:TestPoint_Pad_D1.0mm"
+		(property "Footprint" "Personal-Library:TestPoint_Pad_D1.0mm"
 			(at 161.29 166.37 0)
 			(effects
@@
 			)
 		)
-		(property "Footprint" "TestPoint:TestPoint_Pad_D1.0mm"
+		(property "Footprint" "Personal-Library:TestPoint_Pad_D1.0mm"
 			(at 160.02 171.45 0)
 			(effects
@@
 			)
 		)
-		(property "Footprint" "TestPoint:TestPoint_Pad_D1.0mm"
+		(property "Footprint" "Personal-Library:TestPoint_Pad_D1.0mm"
 			(at 160.02 181.61 0)
 			(effects
@@
 			)
 		)
-		(property "Footprint" "TestPoint:TestPoint_Pad_D1.0mm"
+		(property "Footprint" "Personal-Library:TestPoint_Pad_D1.0mm"
 			(at 160.02 176.53 0)
 			(effects
@@
 			)
 		)
-		(property "Footprint" "TestPoint:TestPoint_Pad_D1.0mm"
+		(property "Footprint" "Personal-Library:TestPoint_Pad_D1.0mm"
 			(at 160.02 186.69 0)
 			(effects
